File: esp32-smart-speaker-schema/wavelet_mini.kicad_sch (KiCad schematic)
At the start: 0 parts

Commit message: Fixed a few bugs for the Wavelet Regular and Max Refactored Codebase
Other:
- company: (none) -> Semire Designs
- title: (none) -> Wavelet Speaker
Changed lines of the file:
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@@
 	(generator_version "9.0")
 	(paper "A4")
+	(title_block
+		(title "Wavelet Speaker")
+		(date "2026-03-12")
+		(rev "1.0.0")
+		(company "Semire Designs")
+		(comment 1 "Available in Mini, Regular, Max")
+	)
 )
